File: pcb/null-city-badge.kicad_sch (KiCad schematic)
At the start: 139 parts, among them J1 USB_C_Receptacle_USB2.0_16P, J10 Conn_01x10_Pin, J11 Conn_Coaxial_Small, J12 Conn_01x07_Pin, J2 Conn_01x02_Pin, J3 Conn_01x06_Pin, J4 Conn_01x24_Socket, J5 Conn_Coaxial_Small, J6 Conn_01x06_Pin, J7 Conn_01x06_Pin, J8 Conn_01x06_Pin, J9 Conn_01x10_Pin, Q1 SS8050, Q2 SS8050, Q3 IRLML0030, Q4 AO3401A, Q5 SS8050, U1 ESP32-S3-WROOM-1, U10 TCA9534, U11 CORE1262-868M, U12 ME6211C33M5, U13 CC1101RGP, U14 ME6211C33M5, U2 CP2102N-Axx-xQFN28, U3 SE050C2HQ1_Z01SDZ, U4 MCP73831-2-MC, U5 ME6211C33M5, U6 ME6211C33M5, U7 NS4168, U8 74125, U9 ME6211C33M5, Y2 26Mhz

Commit message: feat: main board with sub ghz and audio modules, remove lora and sdcard
Parts:
- removed C24, C27, C28, C32, C34, C37, C39, C41, C43, C44: 100n, Capacitor_SMD:C_0402_1005Metric, symbol Device:C
- removed C25, C26, C30, C31, C33, C36, C38, C40, C42: 10U, Capacitor_SMD:C_0402_1005Metric, symbol Device:C
- removed C29: 22U, Capacitor_SMD:C_0402_1005Metric, symbol Device:C
- removed C45, C46: 27p, Capacitor_SMD:C_0402_1005Metric, symbol Device:C
- removed C48, C53: 220p, Capacitor_SMD:C_0402_1005Metric, symbol Device:C
- removed C49, C50: 3.9p, Capacitor_SMD:C_0402_1005Metric, symbol Device:C
- removed C51: 8.2p, Capacitor_SMD:C_0402_1005Metric, symbol Device:C
- removed C52: 5.6p, Capacitor_SMD:C_0402_1005Metric, symbol Device:C
- removed J11, J5: Conn_Coaxial_Small, Connector_Coaxial:SMA_Amphenol_901-143_Horizontal, symbol Connector:Conn_Coaxial_Small
- removed J12: Conn_01x07_Pin, Connector_PinHeader_2.54mm:PinHeader_1x07_P2.54mm_Vertical, symbol Connector:Conn_01x07_Pin
- removed J6, J7: Conn_01x06_Pin, Connector_PinHeader_2.54mm:PinHeader_1x06_P2.54mm_Vertical, symbol Connector:Conn_01x06_Pin
- removed J9: Conn_01x10_Pin, Connector_PinHeader_2.54mm:PinHeader_1x10_P2.54mm_Vertical, symbol Connector:Conn_01x10_Pin
- removed L4: 22nH, Inductor_SMD:L_0402_1005Metric, symbol Device:L
- removed L5, L6, L7: 27nH, Inductor_SMD:L_0402_1005Metric, symbol Device:L
- removed MICRO_SD1: TF-01A, NIP_MOD:TF-01A, symbol PCM_NIP_MOD:TF-01A
- removed MK1, MK2: ICS-43434, Sensor_Audio:InvenSense_ICS-43434-6_3.5x2.65mm, symbol Sensor_Audio:ICS-43434
- removed R24: 1K, Resistor_SMD:R_0402_1005Metric, symbol Device:R
- removed R25, R26, R27, R28: 2K2, Resistor_SMD:R_0402_1005Metric, symbol Device:R
- removed R29: 56K, Resistor_SMD:R_0402_1005Metric, symbol Device:R
- removed TP1: SP+, Connector_Pin:Pin_D1.3mm_L11.0mm, symbol Connector:TestPoint
- removed TP2: SP-, Connector_Pin:Pin_D1.3mm_L11.0mm, symbol Connector:TestPoint
- removed U11: CORE1262-868M, NIP_MOD:XCVR_CORE1262-868M, symbol PCM_NIP_MOD:CORE1262-868M
- removed U12, U14, U6, U9: ME6211C33M5, Package_TO_SOT_SMD:SOT-23-5, symbol Regulator_Linear:ME6211C33M5
- removed U13: CC1101RGP, NIP_MOD:QFN50P400X400X100-21N, symbol PCM_CC1101RGP:CC1101RGP
- removed U7: NS4168, Package_SO:SOIC-8-1EP_3.9x4.9mm_P1.27mm_EP2.29x3mm, symbol PCM_NIP_MOD:NS4168
- removed U8: 74125, Package_SO:TSSOP-14_4.4x5mm_P0.65mm, symbol 74xx_IEEE:74125
- removed Y2: 26Mhz, Crystal:Crystal_SMD_3225-4Pin_3.2x2.5mm, symbol Device:Crystal_GND24_Small
- C2: value 1OOn -> 100n
- J2: footprint Connector_JST:JST_GH_SM02B-GHS-TB_1x02-1MP_P1.25mm_Horizontal -> Connector_JST:JST_PH_S2B-PH-SM4-TB_1x02-1MP_P2.00mm_Horizontal
- PB1, PB2, PB3, PB4, PB5, PB6: footprint Button_Switch_SMD:SW_SPST_B3SL-1002P -> Button_Switch_SMD:SW_Push_1TS009xxxx-xxxx-xxxx_6x6x5mm
Connections:
- net at C20.1, Q4.1 (G), Q5.3 (C)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: now also ON/OFF_PB1.1; no longer ON/OFF_PB1.2
- net GND renamed GND1
- net GND1: now also ON/OFF_PB1.2, U4.9 (EP); no longer ON/OFF_PB1.1
Other:
- added sheet CC1101 MODULE (CC1101_MOD.kicad_sch)
- added sheet LORA MODULE (LORA_MOD.kicad_sch)
- added sheet SD CARD MODULE (SDCARD_MOD.kicad_sch)
- added sheet SOUND MODULE (SOUND_MOD.kicad_sch)
- moved on the sheet: BOOT1, C1, C10, C11, C12, C13, C14, C15, C16, C17, C18, C19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
