File: pcb/SOUND_MOD.kicad_sch (KiCad schematic)
At the start: 14 parts, among them J6 Conn_01x07_Pin, U6 ME6211C33M5, U7 NS4168

Commit message: feat: final file for production with panel adjustment
Parts:
- added C31: 22U, Capacitor_SMD:C_0402_1005Metric, symbol Device:C
Connections:
- net at TP1.1: now also C31.1; no longer U7.8 (VOP)
- new net: C31.2, U7.8 (VOP)
Other:
- moved on the sheet: TP1
Changed lines of the file:
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@@
+	(wire
+		(pts
+			(xy 175.26 57.15) (xy 175.26 62.23)
+		)
+		(stroke
+			(width 0)
+			(type default)
+		)
+	)
 	(wire
 		(pts
@@
 	)
 	(symbol
+		(lib_id "Device:C")
+		(at 175.26 53.34 0)
+		(unit 1)
+		(exclude_from_sim no)
+		(in_bom yes)
+		(on_board yes)
+		(dnp no)
+		(fields_autoplaced yes)
+		(property "Reference" "C31"
+			(at 179.07 52.0699 0)
+			(effects
+				(font
+					(size 1.27 1.27)
+				)
+				(justify left)
+			)
+		)
+		(property "Value" "22U"
+			(at 179.07 54.6099 0)
+			(effects
+				(font
+					(size 1.27 1.27)
+				)
+				(justify left)
+			)
+		)
+		(property "Footprint" "Capacitor_SMD:C_0402_1005Metric"
+			(at 176.2252 57.15 0)
+			(effects
+				(font
+					(size 1.27 1.27)
+				)
+				(hide yes)
+			)
+		)
+		(property "Datasheet" "~"
+			(at 175.26 53.34 0)
+			(effects
+				(font
+					(size 1.27 1.27)
+				)
+				(hide yes)
+			)
+		)
+		(property "Description" "Unpolarized capacitor"
+			(at 175.26 53.34 0)
+			(effects
+				(font
+					(size 1.27 1.27)
+				)
+				(hide yes)
+			)
+		)
+		(pin "2"
+		)
+		(pin "1"
+		)
+		(instances
+			(project "null-city-badge"
+				(path "/96a9ebd7-4f87-4060-87a7-f00d27473ddc/8c5168c8-f359-473b-9459-5b246b7098e5"
+					(reference "C31")
+					(unit 1)
+				)
+			)
+		)
+	)
+	(symbol
 		(lib_id "PCM_NIP_MOD:NS4168")
 		(at 165.1 66.04 0)
@@
 	(symbol
 		(lib_id "Connector:TestPoint")
-		(at 175.26 62.23 0)
+		(at 175.26 49.53 0)
 		(unit 1)
 		(exclude_from_sim no)
@@
 		(fields_autoplaced yes)
 		(property "Reference" "TP1"
-			(at 177.8 57.6579 0)
+			(at 177.8 44.9579 0)
 			(effects
 				(font
@@
 		)
 		(property "Value" "SP+"
-			(at 177.8 60.1979 0)
+			(at 177.8 47.4979 0)
 			(effects
 				(font
@@
 		)
 		(property "Footprint" "Connector_Pin:Pin_D1.3mm_L11.0mm"
-			(at 180.34 62.23 0)
+			(at 180.34 49.53 0)
 			(effects
 				(font
@@
 		)
 		(property "Datasheet" "~"
-			(at 180.34 62.23 0)
+			(at 180.34 49.53 0)
 			(effects
 				(font
@@
 		)
 		(property "Description" "test point"
-			(at 175.26 62.23 0)
-			(effects
-				(font
+			(at 175.26 49.53 0)
+			(effects
+				(font
