File: pcb/null-city-badge.kicad_pcb (KiCad board)
At the start: 2 copper layers, 76.6 x 141.1 mm, 189 parts, among them J1 USB_C_Receptacle_USB2.0_16P, J10 Conn_01x10_Pin, J11 Conn_Coaxial_Small, J12 Conn_01x07_Pin, J2 Conn_01x02_Pin, J3 Conn_01x04_Pin, J4 Conn_01x24_Socket, J6 Conn_01x07_Pin, J8 Conn_01x06_Pin, Q1 SS8050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

Commit message: feat: final file for production with panel adjustment
Parts:
- added C31: 10U, Capacitor_SMD:C_0402_1005Metric, B.Cu at (91.2, 171.6)
- moved C41 1.57 mm to (70.5, 157.8)
- moved U13 1.57 mm to (64.3, 165.3)
- moved C46 1.57 mm to (61.1, 171.0)
- moved C48 1.57 mm to (60.4, 168.6)
- moved C49 1.57 mm to (60.4, 163.4)
- moved C50 1.57 mm to (60.4, 166.6)
- moved C53 1.57 mm to (53.3, 165.6)
- moved G*** 1.57 mm to (56.7, 161.8)
- moved G*** 1.57 mm to (56.9, 169.4)
- moved J11 1.57 mm to (47.9, 165.6)
- moved L4 1.57 mm to (60.4, 167.6)
- moved L5 1.57 mm to (60.4, 164.6)
- moved L6 1.57 mm to (59.3, 165.6)
- moved L7 1.57 mm to (56.3, 165.6)
- moved R29 1.57 mm to (63.1, 161.9)
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Connections:
- TP1 pad 1: Net-(U7-VOP) -> Net-(C31-Pad1)
Routing:
- net Net-(U7-VOP): track 25.8 -> 1.76 mm
- net Net-(C31-Pad1): track 0.00 -> 23.1 mm
Other:
- outline, holes or cut-outs redrawn
